File: rechargeble_pack.kicad_sch (KiCad schematic)
At the start: 42 parts, among them J1 Out, J2 LiPo, J3 DC IN, Q1 SIA453, Q2 BC857, Q6 BC847, Q7 BC857, U1 TP4056, U2 TPS61041

Commit message: Schematics fix
Schematics values fix
Parts:
- L1, L2, L3: value 10mH -> 10µH
Other:
- moved on the sheet: C14
Changed lines of the file:
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@@
 	)
 	(junction
-		(at 259.08 73.66)
+		(at 31.75 50.8)
 		(diameter 0)
 		(color 0 0 0 0)
 	)
 	(junction
-		(at 256.54 118.11)
+		(at 259.08 73.66)
 		(diameter 0)
 		(color 0 0 0 0)
 	)
 	(junction
-		(at 267.97 73.66)
+		(at 256.54 118.11)
 		(diameter 0)
 		(color 0 0 0 0)
 	)
 	(junction
-		(at 54.61 50.8)
+		(at 267.97 73.66)
 		(diameter 0)
 		(color 0 0 0 0)
@@
 	(wire
 		(pts
+			(xy 31.75 50.8) (xy 58.42 50.8)
+		)
+		(stroke
+			(width 0)
+			(type default)
+		)
+	)
+	(wire
+		(pts
 			(xy 186.69 107.95) (xy 186.69 118.11)
 		)
@@
 	(wire
 		(pts
+			(xy 27.94 45.72) (xy 27.94 50.8)
+		)
+		(stroke
+			(width 0)
+			(type default)
+		)
+	)
+	(wire
+		(pts
 			(xy 247.65 118.11) (xy 256.54 118.11)
 		)
@@
 	(wire
 		(pts
-			(xy 88.9 78.74) (xy 87.63 78.74)
+			(xy 27.94 50.8) (xy 31.75 50.8)
 		)
 		(stroke
@@
 	(wire
 		(pts
-			(xy 267.97 85.09) (xy 271.78 85.09)
+			(xy 88.9 78.74) (xy 87.63 78.74)
 		)
 		(stroke
@@
 	(wire
 		(pts
-			(xy 31.75 63.5) (xy 31.75 73.66)
+			(xy 267.97 85.09) (xy 271.78 85.09)
 		)
 		(stroke
@@
 	(wire
 		(pts
-			(xy 58.42 74.93) (xy 58.42 50.8)
+			(xy 31.75 63.5) (xy 31.75 73.66)
 		)
 		(stroke
@@
 	(wire
 		(pts
-			(xy 54.61 50.8) (xy 58.42 50.8)
-		)
-		(stroke
-			(width 0)
-			(type default)
-		)
-	)
-	(wire
-		(pts
 			(xy 181.61 118.11) (xy 186.69 118.11)
 		)
@@
 	(wire
 		(pts
-			(xy 173.99 149.86) (xy 165.1 149.86)
+			(xy 173.99 149.86) (xy 176.53 149.86)
 		)
 		(stroke
@@
 	(wire
 		(pts
-			(xy 31.75 50.8) (xy 54.61 50.8)
-		)
-		(stroke
-			(width 0)
-			(type default)
-		)
-	)
-	(wire
-		(pts
 			(xy 173.99 119.38) (xy 173.99 118.11)
 		)
@@
 	(wire
 		(pts
+			(xy 58.42 58.42) (xy 58.42 57.15)
+		)
+		(stroke
+			(width 0)
+			(type default)
+		)
+	)
+	(wire
+		(pts
 			(xy 58.42 50.8) (xy 71.12 50.8)
 		)
@@
 	)
 	(label "OUT_EN"
-		(at 165.1 149.86 0)
+		(at 176.53 149.86 0)
 		(effects
 			(font
@@
 			)
 		)
-		(property "Value" "10mH"
+		(property "Value" "10µH"
 			(at 262.89 21.59 90)
 			(effects
@@
 	(symbol
 		(lib_id "power:GND")
-		(at 58.42 82.55 0)
+		(at 58.42 57.15 0)
 		(unit 1)
 		(exclude_from_sim no)
@@
 		(fields_autoplaced yes)
 		(property "Reference" "#PWR031"
-			(at 58.42 88.9 0)
+			(at 58.42 63.5 0)
 			(effects
 				(font
@@
 		)
 		(property "Value" "GND"
-			(at 58.42 87.63 0)
+			(at 58.42 62.23 0)
 			(effects
 				(font
@@
 		)
 		(property "Footprint" ""
-			(at 58.42 82.55 0)
+			(at 58.42 57.15 0)
 			(effects
 				(font
@@
 		)
 		(property "Datasheet" ""
-			(at 58.42 82.55 0)
+			(at 58.42 57.15 0)
 			(effects
 				(font
@@
 		)
 		(property "Description" "Power symbol creates a global label with name \"GND\" , ground"
-			(at 58.42 82.55 0)
+			(at 58.42 57.15 0)
 			(effects
 				(font
@@
 	(symbol
 		(lib_id "Device:C")
-		(at 58.42 78.74 0)
+		(at 58.42 54.61 0)
 		(unit 1)
 		(exclude_from_sim no)
@@
 		(fields_autoplaced yes)
 		(property "Reference" "C14"
-			(at 62.23 77.4699 0)
+			(at 62.23 53.3399 0)
 			(effects
 				(font
@@
 		)
 		(property "Value" "100nF"
-			(at 62.23 80.0099 0)
+			(at 62.23 55.8799 0)
 			(effects
 				(font
@@
 		)
 		(property "Footprint" "Capacitor_SMD:C_0805_2012Metric"
-			(at 59.3852 82.55 0)
+			(at 59.3852 58.42 0)
 			(effects
 				(font
@@
 		)
 		(property "Datasheet" "~"
-			(at 58.42 78.74 0)
+			(at 58.42 54.61 0)
 			(effects
 				(font
@@
 		)
 		(property "Description" "Unpolarized capacitor"
-			(at 58.42 78.74 0)
+			(at 58.42 54.61 0)
 			(effects
 				(font
@@
 	(symbol
 		(lib_id "power:VBUS")
-		(at 54.61 50.8 0)
+		(at 27.94 45.72 0)
 		(unit 1)
 		(exclude_from_sim no)
@@
 		(fields_autoplaced yes)
 		(property "Reference" "#PWR030"
-			(at 54.61 54.61 0)
+			(at 27.94 49.53 0)
 			(effects
 				(font
@@
 		)
 		(property "Value" "VBUS"
-			(at 54.61 45.72 0)
+			(at 27.94 40.64 0)
 			(effects
 				(font
@@
 		)
 		(property "Footprint" ""
-			(at 54.61 50.8 0)
+			(at 27.94 45.72 0)
 			(effects
 				(font
@@
 		)
 		(property "Datasheet" ""
-			(at 54.61 50.8 0)
+			(at 27.94 45.72 0)
 			(effects
 				(font
@@
 		)
 		(property "Description" "Power symbol creates a global label with name \"VBUS\""
-			(at 54.61 50.8 0)
+			(at 27.94 45.72 0)
 			(effects
 				(font
@@
 			)
 		)
-		(property "Value" "10mH"
+		(property "Value" "10µH"
 			(at 199.39 115.57 90)
 			(effects
@@
 			)
 		)
-		(property "Value" "10mH"
+		(property "Value" "10µH"
 			(at 262.89 115.57 90)
 			(effects

Commit message: fix mosfet
Parts:
- Q1: value SIA453 -> IRLML6402
Other:
- moved on the sheet: Q1, R2
Changed lines of the file:
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@@
 	)
 	(junction
-		(at 246.38 81.28)
-		(diameter 0)
-		(color 0 0 0 0)
-	)
-	(junction
 		(at 173.99 118.11)
 		(diameter 0)
@@
 	)
 	(junction
-		(at 248.92 24.13)
+		(at 236.22 33.02)
 		(diameter 0)
 		(color 0 0 0 0)
 	)
 	(junction
-		(at 241.3 33.02)
+		(at 248.92 24.13)
 		(diameter 0)
 		(color 0 0 0 0)
@@
 	(wire
 		(pts
-			(xy 220.98 21.59) (xy 220.98 24.13)
+			(xy 220.98 22.86) (xy 220.98 21.59)
 		)
 		(stroke
@@
 	(wire
 		(pts
+			(xy 246.38 92.71) (xy 246.38 93.98)
+		)
+		(stroke
+			(width 0)
+			(type default)
+		)
+	)
+	(wire
+		(pts
 			(xy 71.12 73.66) (xy 71.12 66.04)
 		)
@@
 	(wire
 		(pts
-			(xy 248.92 24.13) (xy 246.38 24.13)
+			(xy 250.19 81.28) (xy 246.38 81.28)
+		)
+		(stroke
+			(width 0)
+			(type default)
+		)
+	)
+	(wire
+		(pts
+			(xy 248.92 22.86) (xy 241.3 22.86)
 		)
 		(stroke
@@
 	(wire
 		(pts
-			(xy 246.38 81.28) (xy 246.38 82.55)
+			(xy 220.98 22.86) (xy 231.14 22.86)
 		)
 		(stroke
@@
 	(wire
 		(pts
-			(xy 220.98 24.13) (xy 236.22 24.13)
+			(xy 240.03 73.66) (xy 246.38 73.66)
 		)
 		(stroke
@@
 	(wire
 		(pts
-			(xy 240.03 73.66) (xy 246.38 73.66)
+			(xy 267.97 78.74) (xy 267.97 85.09)
 		)
 		(stroke
@@
 	(wire
 		(pts
-			(xy 267.97 78.74) (xy 267.97 85.09)
+			(xy 257.81 24.13) (xy 259.08 24.13)
 		)
 		(stroke
@@
 	(wire
 		(pts
-			(xy 257.81 24.13) (xy 259.08 24.13)
+			(xy 248.92 29.21) (xy 248.92 24.13)
 		)
 		(stroke
@@
 	(wire
 		(pts
-			(xy 248.92 29.21) (xy 248.92 24.13)
+			(xy 223.52 73.66) (xy 223.52 78.74)
 		)
 		(stroke
@@
 	(wire
 		(pts
-			(xy 223.52 73.66) (xy 223.52 78.74)
+			(xy 266.7 93.98) (xy 266.7 76.2)
 		)
 		(stroke
@@
 	(wire
 		(pts
-			(xy 266.7 93.98) (xy 266.7 76.2)
+			(xy 250.19 92.71) (xy 246.38 92.71)
 		)
 		(stroke
@@
 	(wire
 		(pts
+			(xy 248.92 22.86) (xy 248.92 24.13)
+		)
+		(stroke
+			(width 0)
+			(type default)
+		)
+	)
+	(wire
+		(pts
 			(xy 237.49 133.35) (xy 247.65 133.35)
 		)
@@
 	(wire
 		(pts
-			(xy 241.3 33.02) (xy 241.3 31.75)
+			(xy 236.22 33.02) (xy 236.22 30.48)
 		)
 		(stroke
@@
 	(wire
 		(pts
+			(xy 250.19 82.55) (xy 250.19 81.28)
+		)
+		(stroke
+			(width 0)
+			(type default)
+		)
+	)
+	(wire
+		(pts
 			(xy 181.61 125.73) (xy 181.61 118.11)
 		)
@@
 	(wire
 		(pts
+			(xy 236.22 33.02) (xy 241.3 33.02)
+		)
+		(stroke
+			(width 0)
+			(type default)
+		)
+	)
+	(wire
+		(pts
 			(xy 133.35 72.39) (xy 133.35 60.96)
 		)
@@
 	(wire
 		(pts
-			(xy 246.38 88.9) (xy 246.38 93.98)
+			(xy 250.19 90.17) (xy 250.19 92.71)
 		)
 		(stroke
@@
 	(wire
 		(pts
-			(xy 220.98 33.02) (xy 241.3 33.02)
+			(xy 220.98 33.02) (xy 236.22 33.02)
 		)
 		(stroke
@@
 	(symbol
 		(lib_id "Simulation_SPICE:PMOS")
-		(at 241.3 26.67 90)
+		(at 236.22 25.4 90)
 		(unit 1)
 		(exclude_from_sim no)
@@
 		(on_board yes)
 		(dnp no)
-		(fields_autoplaced yes)
 		(property "Reference" "Q1"
-			(at 241.3 17.78 90)
+			(at 236.22 16.51 90)
 			(effects
 				(font
@@
 			)
 		)
-		(property "Value" "SIA453"
-			(at 241.3 20.32 90)
+		(property "Value" "IRLML6402"
+			(at 236.22 19.05 90)
 			(effects
 				(font
@@
 		)
 		(property "Footprint" "Package_TO_SOT_SMD:SOT-23"
-			(at 238.76 21.59 0)
+			(at 233.68 20.32 0)
 			(effects
 				(font
@@
 			)
 		)
-		(property "Datasheet" "https://ngspice.sourceforge.io/docs/ngspice-html-manual/manual.xhtml#cha_MOSFETs"
-			(at 254 26.67 0)
+		(property "Datasheet" ""
+			(at 248.92 25.4 0)
 			(effects
 				(font
@@
 		)
 		(property "Description" "P-MOSFET transistor, drain/source/gate"
-			(at 241.3 26.67 0)
+			(at 236.22 25.4 0)
 			(effects
 				(font
@@
 		)
 		(property "Sim.Device" "PMOS"
-			(at 258.445 26.67 0)
+			(at 253.365 25.4 0)
 			(effects
 				(font
@@
 		)
 		(property "Sim.Type" "VDMOS"
-			(at 260.35 26.67 0)
+			(at 255.27 25.4 0)
 			(effects
 				(font
@@
 		)
 		(property "Sim.Pins" "1=D 2=G 3=S"
-			(at 256.54 26.67 0)
+			(at 230.124 42.164 90)
 			(effects
 				(font
@@
 	(symbol
 		(lib_id "Device:R")
-		(at 246.38 85.09 0)
+		(at 250.19 86.36 0)
 		(unit 1)
 		(exclude_from_sim no)
@@
 		(fields_autoplaced yes)
 		(property "Reference" "R2"
-			(at 248.92 83.8199 0)
+			(at 252.73 85.0899 0)
 			(effects
 				(font
@@
 		)
 		(property "Value" "10R"
-			(at 248.92 86.3599 0)
+			(at 252.73 87.6299 0)
 			(effects
 				(font
@@
 		)
 		(property "Footprint" "Resistor_SMD:R_0805_2012Metric"
-			(at 244.602 85.09 90)
+			(at 248.412 86.36 90)
 			(effects
 				(font
@@
 		)
 		(property "Datasheet" "~"
-			(at 246.38 85.09 0)
+			(at 250.19 86.36 0)
 			(effects
 				(font
@@
 		)
 		(property "Description" "Resistor"
-			(at 246.38 85.09 0)
+			(at 250.19 86.36 0)
 			(effects
 				(font
